Commit message: Save migration-ready draft: MiniMax LLM patches and runtime fixes.
Include IsaacGymEnvs sources, Franka URDF path fix, RRT 2D coerce, RTX4090 JIT workaround, and troubleshooting notes. API secrets left empty.

Co-authored-by: Cursor <cursoragent@cursor.com>

File: Agent_asset/franka_description/robots/franka_panda.urdf (robot description, URDF)
Before this commit: robot panda, 11 links, 10 joints
Links:
- link panda_hand: geometry collision mesh filename=../meshes/collision/hand.obj; visual mesh filename=../meshes/visual/hand.dae
- link panda_leftfinger: geometry collision mesh filename=../meshes/collision/finger.obj; visual mesh filename=../meshes/visual/finger.dae
- link panda_link0: geometry collision mesh filename=../meshes/collision/link0.obj; visual mesh filename=../meshes/visual/link0.dae
- link panda_link1: geometry collision mesh filename=../meshes/collision/link1.obj; visual mesh filename=../meshes/visual/link1.dae
- link panda_link2: geometry collision mesh filename=../meshes/collision/link2.obj; visual mesh filename=../meshes/visual/link2.dae
- link panda_link3: geometry collision mesh filename=../meshes/collision/link3.obj; visual mesh filename=../meshes/visual/link3.dae
- link panda_link4: geometry collision mesh filename=../meshes/collision/link4.obj; visual mesh filename=../meshes/visual/link4.dae
- link panda_link5: geometry collision mesh filename=../meshes/collision/link5.obj; visual mesh filename=../meshes/visual/link5.dae
- link panda_link6: geometry collision mesh filename=../meshes/collision/link6.obj; visual mesh filename=../meshes/visual/link6.dae
- link panda_link7: geometry collision mesh filename=../meshes/collision/link7.obj; visual mesh filename=../meshes/visual/link7.dae
- link panda_rightfinger: geometry collision mesh filename=../meshes/collision/finger.obj; visual mesh filename=../meshes/visual/finger.dae
